File: roompatch/RoomControllerConnector.kicad_sch (KiCad schematic)
At the start: 1 part, among them J2 ROOM CONTROLLER

Commit message: 20260607A
Parts:
- J2: footprint Connector_IDC:IDC-Header_2x10_P2.54mm_Horizontal -> Connector_IDC:IDC-Header_2x10_P2.54mm_Vertical
Connections:
- net 12V renamed POWER
- net INPUT_ALARM: no longer names the net of J2.8 (Pin_8)
- net INPUT_MAG1 renamed SOUNDER
- net INPUT_MAG2 renamed STROBE
- net INPUT_MAG3: no longer names the net of J2.3 (Pin_3)
- net INPUT_PIR1: no longer names the net of J2.5 (Pin_5)
- net INPUT_PIR1: no longer J2.19 (Pin_19)
- net INPUT_PIR2: no longer names the net of J2.7 (Pin_7)
- net INPUT_PIR2: no longer J2.18 (Pin_18)
- net INPUT_SAFETY renamed INPUT_DOOR
- new net INPUT_FIRE: J2.19 (Pin_19)
- new net INPUT_PIR: J2.18 (Pin_18)
- no-connect marks 0 -> 4
Changed lines of the file:
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@@
 (kicad_sch
-	(version 20250114)
+	(version 20260306)
 	(generator "eeschema")
-	(generator_version "9.0")
+	(generator_version "10.0")
 	(paper "A4")
+	(no_connect
+		(at 107.95 77.47)
+	)
+	(no_connect
+		(at 107.95 82.55)
+	)
+	(no_connect
+		(at 107.95 90.17)
+	)
+	(no_connect
+		(at 107.95 87.63)
+	)
 	(wire
 		(pts
-			(xy 107.95 90.17) (xy 104.14 90.17)
+			(xy 107.95 92.71) (xy 106.68 92.71)
 		)
 		(stroke
@@
 	(wire
 		(pts
-			(xy 107.95 92.71) (xy 106.68 92.71)
+			(xy 104.14 95.25) (xy 107.95 95.25)
 		)
 		(stroke
@@
 		)
 	)
-	(wire
-		(pts
-			(xy 104.14 95.25) (xy 107.95 95.25)
-		)
-		(stroke
-			(width 0)
-			(type default)
-		)
-	)
 	(hierarchical_label "RSP_DATA+"
 		(shape input)
@@
 		)
 	)
-	(hierarchical_label "INPUT_PIR2"
+	(hierarchical_label "INPUT_TAMP2"
+		(shape input)
+		(at 107.95 85.09 180)
+		(effects
+			(font
+				(size 1.27 1.27)
+			)
+			(justify right)
+		)
+	)
+	(hierarchical_label "INPUT_DOOR"
+		(shape input)
+		(at 107.95 74.93 180)
+		(effects
+			(font
+				(size 1.27 1.27)
+			)
+			(justify right)
+		)
+	)
+	(hierarchical_label "SOUNDER"
+		(shape output)
+		(at 120.65 80.01 0)
+		(effects
+			(font
+				(size 1.27 1.27)
+			)
+			(justify left)
+		)
+	)
+	(hierarchical_label "GND"
+		(shape passive)
+		(at 120.65 95.25 0)
+		(effects
+			(font
+				(size 1.27 1.27)
+			)
+			(justify left)
+		)
+	)
+	(hierarchical_label "STROBE"
+		(shape output)
+		(at 120.65 82.55 0)
+		(effects
+			(font
+				(size 1.27 1.27)
+			)
+			(justify left)
+		)
+	)
+	(hierarchical_label "5V"
+		(shape passive)
+		(at 107.95 72.39 180)
+		(effects
+			(font
+				(size 1.27 1.27)
+			)
+			(justify right)
+		)
+	)
+	(hierarchical_label "GND"
+		(shape passive)
+		(at 106.68 92.71 180)
+		(effects
+			(font
+				(size 1.27 1.27)
+			)
+			(justify right)
+		)
+	)
+	(hierarchical_label "INPUT_FIRE"
+		(shape input)
+		(at 120.65 74.93 0)
+		(effects
+			(font
+				(size 1.27 1.27)
+			)
+			(justify left)
+		)
+	)
+	(hierarchical_label "FLOOR_TEMP_DATA"
+		(shape input)
+		(at 120.65 92.71 0)
+		(effects
+			(font
+				(size 1.27 1.27)
+			)
+			(justify left)
+		)
+	)
+	(hierarchical_label "INPUT_TAMP1"
+		(shape input)
+		(at 107.95 80.01 180)
+		(effects
+			(font
+				(size 1.27 1.27)
+			)
+			(justify right)
+		)
+	)
+	(hierarchical_label "INPUT_PIR"
 		(shape input)
 		(at 120.65 77.47 0)
@@
 		)
 	)
-	(hierarchical_label "INPUT_TAMP2"
-		(shape input)
-		(at 107.95 85.09 180)
-		(effects
-			(font
-				(size 1.27 1.27)
-			)
-			(justify right)
-		)
-	)
-	(hierarchical_label "INPUT_MAG2"
-		(shape input)
-		(at 120.65 82.55 0)
-		(effects
-			(font
-				(size 1.27 1.27)
-			)
-			(justify left)
-		)
-	)
-	(hierarchical_label "GND"
-		(shape passive)
-		(at 120.65 95.25 0)
-		(effects
-			(font
-				(size 1.27 1.27)
-			)
-			(justify left)
-		)
-	)
-	(hierarchical_label "INPUT_ALARM"
-		(shape input)
-		(at 104.14 90.17 180)
-		(effects
-			(font
-				(size 1.27 1.27)
-			)
-			(justify right)
-		)
-	)
-	(hierarchical_label "5V"
-		(shape passive)
-		(at 107.95 72.39 180)
-		(effects
-			(font
-				(size 1.27 1.27)
-			)
-			(justify right)
-		)
-	)
-	(hierarchical_label "GND"
-		(shape passive)
-		(at 106.68 92.71 180)
-		(effects
-			(font
-				(size 1.27 1.27)
-			)
-			(justify right)
-		)
-	)
-	(hierarchical_label "FLOOR_TEMP_DATA"
-		(shape input)
-		(at 120.65 92.71 0)
-		(effects
-			(font
-				(size 1.27 1.27)
-			)
-			(justify left)
-		)
-	)
-	(hierarchical_label "INPUT_PIR1"
-		(shape input)
-		(at 120.65 74.93 0)
-		(effects
-			(font
-				(size 1.27 1.27)
-			)
-			(justify left)
-		)
-	)
-	(hierarchical_label "INPUT_TAMP1"
-		(shape input)
-		(at 107.95 80.01 180)
-		(effects
-			(font
-				(size 1.27 1.27)
-			)
-			(justify right)
-		)
-	)
-	(hierarchical_label "INPUT_SAFETY"
-		(shape input)
-		(at 107.95 74.93 180)
-		(effects
-			(font
-				(size 1.27 1.27)
-			)
-			(justify right)
-		)
-	)
 	(hierarchical_label "RSP_DATA-"
 		(shape input)
@@
 		)
 	)
-	(hierarchical_label "INPUT_PIR1"
-		(shape input)
-		(at 107.95 82.55 180)
-		(effects
-			(font
-				(size 1.27 1.27)
-			)
-			(justify right)
-		)
-	)
-	(hierarchical_label "INPUT_MAG1"
-		(shape input)
-		(at 120.65 80.01 0)
-		(effects
-			(font
-				(size 1.27 1.27)
-			)
-			(justify left)
-		)
-	)
-	(hierarchical_label "12V"
+	(hierarchical_label "POWER"
 		(shape passive)
 		(at 120.65 72.39 0)
@@
 			)
 			(justify left)
-		)
-	)
-	(hierarchical_label "INPUT_MAG3"
-		(shape input)
-		(at 107.95 77.47 180)
-		(effects
-			(font
-				(size 1.27 1.27)
-			)
-			(justify right)
-		)
-	)
-	(hierarchical_label "INPUT_PIR2"
-		(shape input)
-		(at 107.95 87.63 180)
-		(effects
-			(font
-				(size 1.27 1.27)
-			)
-			(justify right)
 		)
 	)
@@
 		(at 113.03 82.55 0)
 		(unit 1)
+		(body_style 1)
 		(exclude_from_sim no)
 		(in_bom yes)
 		(on_board yes)
+		(in_pos_files yes)
 		(dnp no)
 		(fields_autoplaced yes)
 		(property "Reference" "J2"
 			(at 114.3 66.04 0)
+			(show_name no)
+			(do_not_autoplace no)
 			(effects
 				(font
@@
 		(property "Value" "ROOM CONTROLLER"
 			(at 114.3 68.58 0)
-			(effects
-				(font
-					(size 1.27 1.27)
-				)
-			)
-		)
-		(property "Footprint" "Connector_IDC:IDC-Header_2x10_P2.54mm_Horizontal"
+			(show_name no)
+			(do_not_autoplace no)
+			(effects
+				(font
+					(size 1.27 1.27)
+				)
+			)
+		)
+		(property "Footprint" "Connector_IDC:IDC-Header_2x10_P2.54mm_Vertical"
 			(at 113.03 82.55 0)
-			(effects
-				(font
-					(size 1.27 1.27)
-				)
-				(hide yes)
-			)
-		)
-		(property "Datasheet" "~"
+			(hide yes)
+			(show_name no)
+			(do_not_autoplace no)
+			(effects
+				(font
+					(size 1.27 1.27)
+				)
+			)
+		)
+		(property "Datasheet" ""
 			(at 113.03 82.55 0)
-			(effects
-				(font
-					(size 1.27 1.27)
-				)
-				(hide yes)
+			(hide yes)
+			(show_name no)
+			(do_not_autoplace no)
+			(effects
+				(font
+					(size 1.27 1.27)
+				)
 			)
 		)
 		(property "Description" "Generic connector, double row, 02x10, counter clockwise pin numbering scheme (similar to DIP package numbering), script generated (kicad-library-utils/schlib/autogen/connector/)"
 			(at 113.03 82.55 0)
-			(effects
-				(font
-					(size 1.27 1.27)
-				)
-				(hide yes)
-			)
-		)
+			(hide yes)
+			(show_name no)
+			(do_not_autoplace no)
+			(effects
+				(font
+					(size 1.27 1.27)
+				)
+			)
+		)

Commit message: 20260607b
Parts:
- removed J2: ROOM CONTROLLER, Connector_IDC:IDC-Header_2x10_P2.54mm_Vertical, symbol Connector_Generic:Conn_02x10_Counter_Clockwise
- added J2: ROOM CONTROLLER, Connector_IDC:IDC-Header_2x07_P2.54mm_Vertical, symbol Connector_Generic:Conn_02x07_Counter_Clockwise
Connections:
- net 5V: now also J2.1 (Pin_1)
- net FLOOR_TEMP_DATA: now also J2.5 (Pin_5)
- net GND: now also J2.6 (Pin_6)
- net INPUT_DOOR: now also J2.2 (Pin_2)
- net INPUT_FIRE: now also J2.13 (Pin_13)
- net INPUT_PIR: now also J2.12 (Pin_12)
- net INPUT_TAMP1: now also J2.3 (Pin_3)
- net INPUT_TAMP2: now also J2.4 (Pin_4)
- net POWER: now also J2.14 (Pin_14)
- net RSP_DATA+: now also J2.8 (Pin_8)
- net RSP_DATA-: now also J2.7 (Pin_7)
- net RSP_RST: now also J2.9 (Pin_9)
- net SOUNDER: now also J2.11 (Pin_11)
- net STROBE: now also J2.10 (Pin_10)
- no-connect marks 4 -> 0
Changed lines of the file:
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@@
 	(generator_version "10.0")
 	(paper "A4")
-	(no_connect
-		(at 107.95 77.47)
-	)
-	(no_connect
-		(at 107.95 82.55)
-	)
-	(no_connect
-		(at 107.95 90.17)
-	)
-	(no_connect
-		(at 107.95 87.63)
-	)
-	(wire
-		(pts
-			(xy 107.95 92.71) (xy 106.68 92.71)
-		)
-		(stroke
-			(width 0)
-			(type default)
-		)
-	)
-	(wire
-		(pts
-			(xy 104.14 95.25) (xy 107.95 95.25)
-		)
-		(stroke
-			(width 0)
-			(type default)
-		)
-	)
 	(hierarchical_label "RSP_DATA+"
 		(shape input)
-		(at 120.65 87.63 0)
+		(at 121.92 62.23 0)
+		(effects
+			(font
+				(size 1.27 1.27)
+			)
+			(justify left)
+		)
+	)
+	(hierarchical_label "INPUT_TAMP2"
+		(shape input)
+		(at 109.22 54.61 180)
+		(effects
+			(font
+				(size 1.27 1.27)
+			)
+			(justify right)
+		)
+	)
+	(hierarchical_label "INPUT_DOOR"
+		(shape input)
+		(at 109.22 49.53 180)
+		(effects
+			(font
+				(size 1.27 1.27)
+			)
+			(justify right)
+		)
+	)
+	(hierarchical_label "SOUNDER"
+		(shape output)
+		(at 121.92 54.61 0)
 		(effects
 			(font
@@
 	(hierarchical_label "GND"
 		(shape passive)
-		(at 104.14 95.25 180)
-		(effects
-			(font
-				(size 1.27 1.27)
-			)
-			(justify right)
-		)
-	)
-	(hierarchical_label "INPUT_TAMP2"
-		(shape input)
-		(at 107.95 85.09 180)
-		(effects
-			(font
-				(size 1.27 1.27)
-			)
-			(justify right)
-		)
-	)
-	(hierarchical_label "INPUT_DOOR"
-		(shape input)
-		(at 107.95 74.93 180)
-		(effects
-			(font
-				(size 1.27 1.27)
-			)
-			(justify right)
-		)
-	)
-	(hierarchical_label "SOUNDER"
-		(shape output)
-		(at 120.65 80.01 0)
-		(effects
-			(font
-				(size 1.27 1.27)
-			)
-			(justify left)
-		)
-	)
-	(hierarchical_label "GND"
-		(shape passive)
-		(at 120.65 95.25 0)
-		(effects
-			(font
-				(size 1.27 1.27)
-			)
-			(justify left)
+		(at 109.22 59.69 180)
+		(effects
+			(font
+				(size 1.27 1.27)
+			)
+			(justify right)
 		)
 	)
 	(hierarchical_label "STROBE"
 		(shape output)
-		(at 120.65 82.55 0)
+		(at 121.92 57.15 0)
 		(effects
 			(font
@@
 	(hierarchical_label "5V"
 		(shape passive)
-		(at 107.95 72.39 180)
-		(effects
-			(font
-				(size 1.27 1.27)
-			)
-			(justify right)
-		)
-	)
-	(hierarchical_label "GND"
-		(shape passive)
-		(at 106.68 92.71 180)
+		(at 109.22 46.99 180)
 		(effects
 			(font
@@
 	(hierarchical_label "INPUT_FIRE"
 		(shape input)
-		(at 120.65 74.93 0)
+		(at 121.92 49.53 0)
 		(effects
 			(font
@@
 	(hierarchical_label "FLOOR_TEMP_DATA"
 		(shape input)
-		(at 120.65 92.71 0)
-		(effects
-			(font
-				(size 1.27 1.27)
-			)
-			(justify left)
+		(at 109.22 57.15 180)
+		(effects
+			(font
+				(size 1.27 1.27)
+			)
+			(justify right)
 		)
 	)
 	(hierarchical_label "INPUT_TAMP1"
 		(shape input)
-		(at 107.95 80.01 180)
+		(at 109.22 52.07 180)
 		(effects
 			(font
@@
 	(hierarchical_label "INPUT_PIR"
 		(shape input)
-		(at 120.65 77.47 0)
+		(at 121.92 52.07 0)
 		(effects
 			(font
@@
 	(hierarchical_label "RSP_DATA-"
 		(shape input)
-		(at 120.65 90.17 0)
-		(effects
-			(font
-				(size 1.27 1.27)
-			)
-			(justify left)
+		(at 109.22 62.23 180)
+		(effects
+			(font
+				(size 1.27 1.27)
+			)
+			(justify right)
 		)
 	)
 	(hierarchical_label "RSP_RST"
 		(shape input)
-		(at 120.65 85.09 0)
+		(at 121.92 59.69 0)
 		(effects
 			(font
@@
 	(hierarchical_label "POWER"
 		(shape passive)
-		(at 120.65 72.39 0)
+		(at 121.92 46.99 0)
 		(effects
 			(font
@@
 	)
 	(symbol
-		(lib_id "Connector_Generic:Conn_02x10_Counter_Clockwise")
-		(at 113.03 82.55 0)
+		(lib_id "Connector_Generic:Conn_02x07_Counter_Clockwise")
+		(at 114.3 54.61 0)
 		(unit 1)
 		(body_style 1)
@@
 		(fields_autoplaced yes)
 		(property "Reference" "J2"
-			(at 114.3 66.04 0)
+			(at 115.57 40.64 0)
 			(show_name no)
 			(do_not_autoplace no)
@@
 		)
 		(property "Value" "ROOM CONTROLLER"
-			(at 114.3 68.58 0)
-			(show_name no)
-			(do_not_autoplace no)
-			(effects
-				(font
-					(size 1.27 1.27)
-				)
-			)
-		)
-		(property "Footprint" "Connector_IDC:IDC-Header_2x10_P2.54mm_Vertical"
-			(at 113.03 82.55 0)
+			(at 115.57 43.18 0)
+			(show_name no)
+			(do_not_autoplace no)
+			(effects
+				(font
+					(size 1.27 1.27)
+				)
+			)
+		)
+		(property "Footprint" "Connector_IDC:IDC-Header_2x07_P2.54mm_Vertical"
+			(at 114.3 54.61 0)
 			(hide yes)
 			(show_name no)
@@
 		)
 		(property "Datasheet" ""
-			(at 113.03 82.55 0)
+			(at 114.3 54.61 0)
 			(hide yes)
 			(show_name no)
@@
 			)
 		)
-		(property "Description" "Generic connector, double row, 02x10, counter clockwise pin numbering scheme (similar to DIP package numbering), script generated (kicad-library-utils/schlib/autogen/connector/)"
-			(at 113.03 82.55 0)
+		(property "Description" "Generic connector, double row, 02x07, counter clockwise pin numbering scheme (similar to DIP package numbering), script generated (kicad-library-utils/schlib/autogen/connector/)"
+			(at 114.3 54.61 0)
 			(hide yes)
 			(show_name no)
@@
 		(pin "14"
 		)
-		(pin "19"
-		)
-		(pin "18"
-		)
-		(pin "17"
-		)
-		(pin "16"
-		)
 		(pin "9"
 		)
-		(pin "15"
-		)
 		(pin "8"
 		)
 		(pin "10"
 		)
-		(pin "20"
-		)
 		(pin "6"
