File: roompatch/roompatch.kicad_pcb (KiCad board)
At the start: 2 copper layers, 160 x 75 mm, 19 parts, among them J1 FLOOR_SENSE, J2 ROOM CONTROLLER

Commit message: 20260607A
Parts:
- removed H16: ~, RWC:RACMultiMountingHoles
- removed IDC3: SENSOR B, TerminalBlock_4Ucon:TerminalBlock_4Ucon_1x04_P3.50mm_Horizontal
- removed JP1: PIR1, Jumper:SolderJumper-2_P1.3mm_Bridged_Pad1.0x1.5mm
- removed JP2: PIR2, Jumper:SolderJumper-2_P1.3mm_Bridged_Pad1.0x1.5mm
- removed JP3: MAG2, Jumper:SolderJumper-2_P1.3mm_Bridged_Pad1.0x1.5mm
- removed JP4: MAG1, Jumper:SolderJumper-2_P1.3mm_Bridged_Pad1.0x1.5mm
- removed RJ45_CENTRAL1: CENTRAL, Connector_RJ:RJ45_HALO_HFJ11-x2450HRL_Horizontal
- removed RJS45_1: RSP, Connector_RJ:RJ45_HALO_HFJ11-x2450HRL_Horizontal
- added CABLETIE10: ~, MountingHole:MountingHole_4mm, F.Cu at (33.1, 89.4)
- added CABLETIE7: ~, MountingHole:MountingHole_4mm, F.Cu at (47.8, 25.7)
- added CABLETIE8: ~, MountingHole:MountingHole_4mm, F.Cu at (47.8, 54.4)
- added CABLETIE9: ~, MountingHole:MountingHole_4mm, F.Cu at (33.1, 80.5)
- added DINMNTA1: ~, MountingHole:MountingHole_5mm, F.Cu at (39.1, 47.4)
- added DINMNTA2: ~, MountingHole:MountingHole_5mm, F.Cu at (73.9, 59.8)
- added DINMNTA3: ~, MountingHole:MountingHole_5mm, F.Cu at (39.1, 72.4)
- added DINMNTB1: ~, MountingHole:MountingHole_5mm, F.Cu at (73.9, 47.3)
- added DINMNTB2: ~, MountingHole:MountingHole_5mm, F.Cu at (39.1, 59.9)
- added DINMNTB3: ~, MountingHole:MountingHole_5mm, F.Cu at (73.9, 72.3)
- added IDC5: BEACON, TerminalBlock_4Ucon:TerminalBlock_4Ucon_1x04_P3.50mm_Horizontal, F.Cu at (62.0, 74.1)
- added IDC6: RSP1, TerminalBlock_4Ucon:TerminalBlock_4Ucon_1x04_P3.50mm_Horizontal, F.Cu at (27.1, 46.8)
- added IDC7: RSP2, TerminalBlock_4Ucon:TerminalBlock_4Ucon_1x04_P3.50mm_Horizontal, F.Cu at (51.5, 36.3)
- added IDC8: C1, TerminalBlock_4Ucon:TerminalBlock_4Ucon_1x04_P3.50mm_Horizontal, F.Cu at (27.1, 74.0)
- added IDC9: C2, TerminalBlock_4Ucon:TerminalBlock_4Ucon_1x04_P3.50mm_Horizontal, F.Cu at (51.5, 63.5)
- IDC1: value PIR1 -> PIR
- IDC2: value SENSOR A -> DOOR
- IDC4: value PIR2 -> FIRE
- J2: footprint Connector_IDC:IDC-Header_2x10_P2.54mm_Horizontal -> Connector_IDC:IDC-Header_2x10_P2.54mm_Vertical
- moved J1 180.8 mm to (51.0, 82.7), turned to -90 degrees
- moved J2 145.7 mm to (84.8, 85.3), turned to -90 degrees
- moved CABLETIE2 137.5 mm to (30.8, 25.7), turned to 90 degrees
- moved IDC2 135.0 mm to (62.0, 46.9)
- moved CABLETIE6 133.4 mm to (30.8, 54.4), turned to 90 degrees
- moved IDC4 112.1 mm to (85.2, 63.6), turned to -90 degrees
- moved IDC1 111.1 mm to (85.2, 36.4), turned to -90 degrees
- moved CABLETIE3 97.3 mm to (64.9, 54.5), turned to 90 degrees
- moved CABLETIE1 97.0 mm to (64.9, 25.8), turned to 90 degrees
- moved CABLETIE5 78.3 mm to (83.3, 25.8), turned to 90 degrees
- moved CABLETIE4 78.2 mm to (83.3, 54.5), turned to 90 degrees
Connections:
- net +12V renamed +POWER
- IDC1 pad 3: INPUT_PIR1 -> INPUT_PIR
- IDC2 pad 2: INPUT_MAG1 -> INPUT_DOOR
- IDC2 pad 4: INPUT_MAG2 -> INPUT_TAMP2
- IDC4 pad 2: INPUT_TAMP2 -> unconnected-(IDC4-Pin_2-Pad2)
- IDC4 pad 3: INPUT_PIR2 -> INPUT_FIRE
- J2 pad 16: INPUT_MAG2 -> STROBE
- J2 pad 17: INPUT_MAG1 -> SOUNDER
- J2 pad 18: INPUT_PIR2 -> INPUT_PIR
- J2 pad 19: INPUT_PIR1 -> INPUT_FIRE
- J2 pad 2: INPUT_SAFETY -> INPUT_DOOR
- J2 pad 3: INPUT_MAG3 -> unconnected-(J2-Pin_3-Pad3)
- J2 pad 5: INPUT_PIR1 -> unconnected-(J2-Pin_5-Pad5)
- J2 pad 7: INPUT_PIR2 -> unconnected-(J2-Pin_7-Pad7)
- J2 pad 8: INPUT_ALARM -> unconnected-(J2-Pin_8-Pad8)
Other:
- board size 160 x 75 mm -> 70 x 75 mm
- board text added: "12V TM2 PIR GND"
- board text added: "DT- N/C N/C GND"
- board text added: "G D +"
- board text added: "PWR DOR FIR PIR"
- board text added: "PWR DOR PWR TM2"
- board text added: "PWR N/C FIR GND"
- board text added: "PWR RST THE DT+"
- board text added: "PWR SND STB GND"
- board text added: "THE SND STB GND"
- board text added: "v1.0 26"
- board text removed: "+ D G"
- board text removed: "G S T +"
- board text removed: "M1 COM M2 COM"
- board text removed: "M3 COM SAF COM"
- board text removed: "v1.0/26"

Commit message: 20260607b
Parts:
- added JP1: THERMO_SIG, Jumper:SolderJumper-2_P1.3mm_Bridged_Pad1.0x1.5mm, F.Cu at (67.7, 95.2)
- J2: footprint Connector_IDC:IDC-Header_2x10_P2.54mm_Vertical -> Connector_IDC:IDC-Header_2x07_P2.54mm_Vertical
- moved CABLETIE10 95.7 mm to (128.7, 93.8)
- moved CABLETIE9 95.6 mm to (128.7, 84.2)
- moved CABLETIE8 83.4 mm to (128.7, 74.7), turned to 0 degrees
- moved CABLETIE5 76.9 mm to (119.1, 93.8), turned to 0 degrees
- moved CABLETIE3 57.8 mm to (119.1, 74.7), turned to 0 degrees
- moved IDC4 57.3 mm to (28.3, 69.5), turned to 90 degrees
- moved IDC1 57.0 mm to (28.3, 37.6), turned to 90 degrees
- moved J2 55.6 mm to (30.0, 94.6), turned to 90 degrees
- moved CABLETIE6 52.7 mm to (68.4, 17.5), turned to 0 degrees
- moved CABLETIE4 46.5 mm to (119.1, 84.2), turned to 0 degrees
- moved IDC6 45.0 mm to (67.5, 27.1), turned to -90 degrees
- moved IDC8 43.2 mm to (67.5, 58.9), turned to -90 degrees
- moved CABLETIE1 38.4 mm to (27.4, 17.5), turned to 0 degrees
- moved IDC5 35.6 mm to (28.3, 85.4)
- moved IDC2 34.4 mm to (28.3, 53.6)
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Connections:
- IDC6 pad 3: THERMOSTAT_SIG -> THERMOSTAT_SIG_IN
- IDC9 pad 1: THERMOSTAT_SIG -> THERMOSTAT_SIG_OUT
- J2 pad 10: GND -> STROBE
- J2 pad 11: GND -> SOUNDER
- J2 pad 12: FLOOR_TEMP_DATA -> INPUT_PIR
- J2 pad 13: RSP_DATA- -> INPUT_FIRE
- J2 pad 14: RSP_DATA+ -> +POWER
- J2 pad 3: unconnected-(J2-Pin_3-Pad3) -> INPUT_TAMP1
- J2 pad 4: INPUT_TAMP1 -> INPUT_TAMP2
- J2 pad 5: unconnected-(J2-Pin_5-Pad5) -> FLOOR_TEMP_DATA
- J2 pad 6: INPUT_TAMP2 -> GND
- J2 pad 7: unconnected-(J2-Pin_7-Pad7) -> RSP_DATA-
- J2 pad 8: unconnected-(J2-Pin_8-Pad8) -> RSP_DATA+
- J2 pad 9: GND -> RSP_RST
Other:
- board size 70 x 75 mm -> 50 x 90 mm
- board text added: "+ D G"
- board text added: "PWR RST THR DT+"
- board text added: "PWR TM1 PIR GND"
- board text added: "THR SND STB GND"
- board text added: "v1.0/26"
- board text removed: "12V TM2 PIR GND"
- board text removed: "G D +"
- board text removed: "PWR RST THE DT+"
- board text removed: "THE SND STB GND"
- board text removed: "v1.0 26"
