File: roompatch/roompatch.kicad_sch (KiCad schematic)
At the start: 17 parts, among them J1 FLOOR_SENSE

Commit message: 20260607A
Parts:
- removed IDC3: SENSOR B, TerminalBlock_4Ucon:TerminalBlock_4Ucon_1x04_P3.50mm_Horizontal, symbol Connector_Generic:Conn_01x04
- removed JP1: PIR1, Jumper:SolderJumper-2_P1.3mm_Bridged_Pad1.0x1.5mm, symbol Jumper:Jumper_2_Bridged
- removed JP2: PIR2, Jumper:SolderJumper-2_P1.3mm_Bridged_Pad1.0x1.5mm, symbol Jumper:Jumper_2_Bridged
- removed JP3: MAG2, Jumper:SolderJumper-2_P1.3mm_Bridged_Pad1.0x1.5mm, symbol Jumper:Jumper_2_Bridged
- removed JP4: MAG1, Jumper:SolderJumper-2_P1.3mm_Bridged_Pad1.0x1.5mm, symbol Jumper:Jumper_2_Bridged
- removed RJS45_1: RSP, Connector_RJ:RJ45_HALO_HFJ11-x2450HRL_Horizontal, symbol Connector:RJ45_Shielded
- added CABLETIE10, CABLETIE11, CABLETIE12, CABLETIE7, CABLETIE8, CABLETIE9: (no value), MountingHole:MountingHole_4mm, symbol JLC PCB Assembly:JLC_PCBA_Tooling_Hole
- added DINMNTA1, DINMNTA2, DINMNTA3, DINMNTB1, DINMNTB2, DINMNTB3: (no value), MountingHole:MountingHole_5mm, symbol JLC PCB Assembly:JLC_PCBA_Tooling_Hole
- added IDC5: BEACON, TerminalBlock_4Ucon:TerminalBlock_4Ucon_1x04_P3.50mm_Horizontal, symbol Connector_Generic:Conn_01x04
- added IDC6: RSP1, TerminalBlock_4Ucon:TerminalBlock_4Ucon_1x04_P3.50mm_Horizontal, symbol Connector_Generic:Conn_01x04
- added IDC7: RSP2, TerminalBlock_4Ucon:TerminalBlock_4Ucon_1x04_P3.50mm_Horizontal, symbol Connector_Generic:Conn_01x04
- CABLETIE1, CABLETIE3, CABLETIE4, CABLETIE5: value ~ -> (none)
- CABLETIE2, CABLETIE6: value ~ -> (none); now in the parts list
- H16: value ~ -> (none); now not fitted
- IDC1: value PIR1 -> PIR
- IDC2: value SENSOR A -> DOOR
- IDC4: value PIR2 -> FIRE
Connections:
- net INPUT_MAG2 is gone; now on net INPUT_TAMP2: IDC2.4 (Pin_4)
- net GND: now also IDC5.4 (Pin_4), IDC7.4 (Pin_4)
- net INPUT_TAMP2: no longer IDC4.2 (Pin_2)
- net RSP_DATA+: now also IDC6.4 (Pin_4)
- net RSP_DATA-: now also IDC7.1 (Pin_1)
- net RSP_RST: now also IDC6.2 (Pin_2)
- net THERMOSTAT_SIG: now also IDC6.3 (Pin_3)
- net +12V renamed +POWER
- net +POWER: now also IDC5.1 (Pin_1), IDC6.1 (Pin_1)
- net INPUT_MAG1 renamed INPUT_DOOR
- net INPUT_PIR1 renamed INPUT_PIR
- net INPUT_PIR2 renamed INPUT_FIRE
- new net SOUNDER: IDC5.2 (Pin_2)
- new net STROBE: IDC5.3 (Pin_3)
- no-connect marks 0 -> 3
Other:
- sheet CentralPatchConnector ports: added INPUT_DOOR, INPUT_FIRE, INPUT_PIR, POWER, SOUNDER, STROBE; removed 12V, 24V, ALARM, MAG, PIR, THERMOSTAT_COM
- sheet RoomControllerConnector ports: added INPUT_DOOR, INPUT_FIRE, INPUT_PIR, POWER, SOUNDER, STROBE; removed 12V, INPUT_ALARM, INPUT_MAG1, INPUT_MAG2, INPUT_MAG3, INPUT_PIR1, INPUT_PIR2, INPUT_SAFETY
- moved on the sheet: IDC4

Commit message: 20260607b
Parts:
- added JP1: THERMO_SIG, Jumper:SolderJumper-2_P1.3mm_Bridged_Pad1.0x1.5mm, symbol Jumper:Jumper_2_Small_Bridged
- CABLETIE10, CABLETIE9: now fitted; now in the parts list
Connections:
- net THERMOSTAT_SIG renamed THERMOSTAT_SIG_IN
- net THERMOSTAT_SIG_IN: now also JP1.2 (B)
- new net THERMOSTAT_SIG_OUT: JP1.1 (A)
Changed lines of the file:
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@@
 	(wire
 		(pts
+			(xy 180.34 72.39) (xy 182.88 72.39)
+		)
+		(stroke
+			(width 0)
+			(type default)
+		)
+	)
+	(wire
+		(pts
 			(xy 80.01 138.43) (xy 82.55 138.43)
 		)
@@
 		)
 	)
+	(global_label "THERMOSTAT_SIG_OUT"
+		(shape output)
+		(at 180.34 72.39 180)
+		(fields_autoplaced yes)
+		(effects
+			(font
+				(size 1.27 1.27)
+			)
+			(justify right)
+		)
+		(property "Intersheetrefs" "${INTERSHEET_REFS}"
+			(at 156.9744 72.39 0)
+			(hide yes)
+			(show_name no)
+			(do_not_autoplace no)
+			(effects
+				(font
+					(size 1.27 1.27)
+				)
+				(justify right)
+			)
+		)
+	)
+	(global_label "THERMOSTAT_SIG_IN"
+		(shape input)
+		(at 187.96 72.39 0)
+		(fields_autoplaced yes)
+		(effects
+			(font
+				(size 1.27 1.27)
+			)
+			(justify left)
+		)
+		(property "Intersheetrefs" "${INTERSHEET_REFS}"
+			(at 209.6323 72.39 0)
+			(hide yes)
+			(show_name no)
+			(do_not_autoplace no)
+			(effects
+				(font
+					(size 1.27 1.27)
+				)
+				(justify left)
+			)
+		)
+	)
 	(global_label "FLOOR_TEMP_DATA"
 		(shape input)
@@
 		)
 	)
-	(global_label "RSP_DATA-"
+	(global_label "THERMOSTAT_SIG_IN"
 		(shape input)
-		(at 80.01 140.97 180)
+		(at 250.19 72.39 180)
 		(fields_autoplaced yes)
 		(effects
@@
 		)
 		(property "Intersheetrefs" "${INTERSHEET_REFS}"
-			(at 66.3205 140.97 0)
+			(at 228.5177 72.39 0)
 			(hide yes)
 			(show_name no)
@@
 		)
 	)
-	(global_label "INPUT_DOOR"
+	(global_label "RSP_DATA-"
 		(shape input)
-		(at 218.44 41.91 180)
+		(at 80.01 140.97 180)
 		(fields_autoplaced yes)
 		(effects
@@
 		)
 		(property "Intersheetrefs" "${INTERSHEET_REFS}"
-			(at 203.9643 41.91 0)
+			(at 66.3205 140.97 0)
 			(hide yes)
 			(show_name no)
@@
 		)
 	)
-	(global_label "INPUT_TAMP2"
+	(global_label "INPUT_DOOR"
 		(shape input)
-		(at 83.82 44.45 180)
+		(at 218.44 41.91 180)
 		(fields_autoplaced yes)
 		(effects
@@
 		)
 		(property "Intersheetrefs" "${INTERSHEET_REFS}"
-			(at 68.3767 44.45 0)
+			(at 203.9643 41.91 0)
 			(hide yes)
 			(show_name no)
@@
 		)
 	)
-	(global_label "THERMOSTAT_SIG"
+	(global_label "INPUT_TAMP2"
 		(shape input)
-		(at 215.9 49.53 180)
+		(at 83.82 44.45 180)
 		(fields_autoplaced yes)
 		(effects
@@
 		)
 		(property "Intersheetrefs" "${INTERSHEET_REFS}"
-			(at 197.1306 49.53 0)
+			(at 68.3767 44.45 0)
 			(hide yes)
 			(show_name no)
@@
 		)
 	)
-	(global_label "SOUNDER"
+	(global_label "THERMOSTAT_SIG_OUT"
 		(shape output)
-		(at 115.57 62.23 180)
+		(at 215.9 49.53 180)
 		(fields_autoplaced yes)
 		(effects
@@
 		)
 		(property "Intersheetrefs" "${INTERSHEET_REFS}"
-			(at 103.6948 62.23 0)
+			(at 192.5344 49.53 0)
 			(hide yes)
 			(show_name no)
@@
 		)
 	)
-	(global_label "INPUT_FIRE"
-		(shape input)
-		(at 123.19 135.89 0)
+	(global_label "SOUNDER"
+		(shape output)
+		(at 115.57 62.23 180)
 		(fields_autoplaced yes)
 		(effects
@@
 				(size 1.27 1.27)
 			)
-			(justify left)
+			(justify right)
 		)
 		(property "Intersheetrefs" "${INTERSHEET_REFS}"
-			(at 137.0005 135.89 0)
+			(at 103.6948 62.23 0)
 			(hide yes)
 			(show_name no)
@@
 					(size 1.27 1.27)
 				)
-				(justify left)
+				(justify right)
 			)
 		)
 	)
-	(global_label "THERMOSTAT_SIG"
+	(global_label "INPUT_FIRE"
 		(shape input)
-		(at 250.19 72.39 180)
+		(at 123.19 135.89 0)
 		(fields_autoplaced yes)
 		(effects
@@
 				(size 1.27 1.27)
 			)
-			(justify right)
+			(justify left)
 		)
 		(property "Intersheetrefs" "${INTERSHEET_REFS}"
-			(at 231.4206 72.39 0)
+			(at 137.0005 135.89 0)
 			(hide yes)
 			(show_name no)
@@
 					(size 1.27 1.27)
 				)
-				(justify right)
+				(justify left)
 			)
 		)
@@
 		(body_style 1)
 		(exclude_from_sim no)
-		(in_bom no)
-		(on_board no)
-		(in_pos_files no)
-		(dnp yes)
+		(in_bom yes)
+		(on_board yes)
+		(in_pos_files yes)
+		(dnp no)
 		(fields_autoplaced yes)
 		(property "Reference" "CABLETIE10"
@@
 	)
 	(symbol
+		(lib_id "Jumper:Jumper_2_Small_Bridged")
+		(at 185.42 72.39 0)
+		(unit 1)
+		(body_style 1)
+		(exclude_from_sim no)
+		(in_bom yes)
+		(on_board yes)
+		(in_pos_files yes)
+		(dnp no)
+		(fields_autoplaced yes)
+		(property "Reference" "JP1"
+			(at 185.42 67.31 0)
+			(show_name no)
+			(do_not_autoplace no)
+			(effects
+				(font
+					(size 1.27 1.27)
+				)
+			)
+		)
+		(property "Value" "THERMO_SIG"
+			(at 185.42 69.85 0)
+			(show_name no)
+			(do_not_autoplace no)
+			(effects
+				(font
+					(size 1.27 1.27)
+				)
+			)
+		)
+		(property "Footprint" "Jumper:SolderJumper-2_P1.3mm_Bridged_Pad1.0x1.5mm"
+			(at 185.42 72.39 0)
+			(hide yes)
+			(show_name no)
+			(do_not_autoplace no)
+			(effects
+				(font
+					(size 1.27 1.27)
+				)
+			)
+		)
+		(property "Datasheet" ""
+			(at 185.42 72.39 0)
+			(hide yes)
+			(show_name no)
+			(do_not_autoplace no)
+			(effects
+				(font
+					(size 1.27 1.27)
+				)
+			)
+		)
+		(property "Description" "Jumper, 2-pole, small symbol, bridged"
+			(at 185.42 72.39 0)
+			(hide yes)
+			(show_name no)
+			(do_not_autoplace no)
+			(effects
+				(font
+					(size 1.27 1.27)
+				)
+			)
+		)
+		(pin "1"
+		)
+		(pin "2"
+		)
+		(instances
+			(project "roompatch"
+				(path "/875b166f-e0fe-493b-829e-f63a6175e073"
+					(reference "JP1")
+					(unit 1)
+				)
+			)
+		)
+	)
+	(symbol
 		(lib_id "JLC PCB Assembly:JLC_PCBA_Tooling_Hole")
 		(at 43.18 80.01 0)
@@
 		(body_style 1)
 		(exclude_from_sim no)
-		(in_bom no)
-		(on_board no)
-		(in_pos_files no)
-		(dnp yes)
+		(in_bom yes)
+		(on_board yes)
+		(in_pos_files yes)
+		(dnp no)
 		(fields_autoplaced yes)
 		(property "Reference" "CABLETIE9"
